Commit message: Basic Motion in RVIZ.

File: dji_m600_sim/urdf/gazebo.xacro (robot description, xacro)
@@ -3,5 +3,5 @@
     <xacro:macro name="base_gazebo">
         <gazebo reference="base_link">
-            <material>Gazebo/Black</material>
+            <material>Gazebo/Blue</material>
         </gazebo>
     </xacro:macro>

File: dji_m600_sim/urdf/links.xacro (robot description, xacro)
@@ -8,7 +8,7 @@
   <xacro:include filename="$(find dji_m600_sim)/urdf/gazebo.xacro" />
   <xacro:macro name="base_link">
-   <link name="base_footprint"/>
+   <link name="world"/>
     <joint name="base_joint" type="fixed">
-      <parent link="base_footprint"/>
+      <parent link="world"/>
       <child link="base_link" />
       <origin xyz="${chassisXoffset} ${chassisYoffset} ${chassisZoffset}" rpy="0 0 0"/>
@@ -17,4 +17,5 @@
       <visual>
         <xacro:box_geometry />
+        <material name="blue" />
       </visual>
       <collision>
