Commit message: Improve multi and moving object. Finished SVD Encore

File: dji_m600_sim/urdf/geometries.xacro (robot description, xacro)
@@ -12,4 +12,10 @@
         </geometry>
 	</xacro:macro>
+    <xacro:macro name="drone_cylinder">
+        <geometry>
+            <cylinder length="${chassisH}" radius="${chassisW/2-0.05}"/>
+        </geometry>
+        <!-- <origin rpy="0 0 0" xyz="0 0 0"/> -->
+    </xacro:macro>
     <xacro:macro name="lidar_geometry">
         <geometry>

File: dji_m600_sim/urdf/links.xacro (robot description, xacro)
@@ -17,10 +17,10 @@
     <link name="vehicle_center_link">
       <visual>
-        <geometry>
-          <mesh filename="file://$(find dji_m600_sim)/meshes/m600.dae" scale="${chassisScale} ${chassisScale} ${chassisScale}"/>
-        </geometry>
+        <!-- <geometry> -->
+          <!-- <mesh filename="file://$(find dji_m600_sim)/meshes/m600.dae" scale="${chassisScale} ${chassisScale} ${chassisScale}"/> -->
+        <!-- </geometry> -->
         <origin rpy="0 0 0" xyz="${chassisMeshXoffset} ${chassisMeshYoffset} ${chassisMeshZoffset}" />
-        <!-- <xacro:box_geometry /> -->
-        <!-- <material name="blue" /> -->
+        <xacro:drone_cylinder />
+        <material name="blue" />
       </visual>
       <collision>

File: dji_m600_sim/urdf/materials.xacro (robot description, xacro)
@@ -21,5 +21,5 @@
     </material>
     <material name="red">
-        <color rgba="0.8 0.0 0.0 1.0"/>
+        <color rgba="1.0 0.0 0.0 1.0"/>
     </material>
     <material name="white">
