Commit message: Add path and M600 Mesh

File: dji_m600_sim/urdf/links.xacro (robot description, xacro)
@@ -16,6 +16,9 @@
     <link name="base_link">
       <visual>
-        <xacro:box_geometry />
-        <material name="blue" />
+        <geometry>
+          <mesh filename="file://$(find dji_m600_sim)/meshes/m600.dae" scale="${chassisScale} ${chassisScale} ${chassisScale}"/>
+        </geometry>
+        <origin rpy="0 0 0" xyz="${chassisMeshXoffset} ${chassisMeshYoffset} ${chassisMeshZoffset}" />
+        <!-- <material name="blue" /> -->
       </visual>
       <collision>

File: dji_m600_sim/urdf/properties.xacro (robot description, xacro)
@@ -16,7 +16,7 @@
     <xacro:property name="chassisIyz" value="0.0"/>
     <xacro:property name="chassisIzz" value="0.0"/>
-    <!-- <xacro:property name="chassisScale" value="0.001"/> -->
-    <!-- <xacro:property name="chassisMeshXoffset" value="-0.125"/>
-    <xacro:property name="chassisMeshYoffset" value="-0.070"/>
-    <xacro:property name="chassisMeshZoffset" value="-0.085"/> -->
+    <xacro:property name="chassisScale" value="1"/>
+    <xacro:property name="chassisMeshXoffset" value="0.000"/>
+    <xacro:property name="chassisMeshYoffset" value="0.000"/>
+    <xacro:property name="chassisMeshZoffset" value="-0.36"/>
 </robot>

Commit message: Parameterize values. Add noise to detection

File: dji_m600_sim/urdf/links.xacro (robot description, xacro)
@@ -16,9 +16,10 @@
     <link name="base_link">
       <visual>
-        <geometry>
-          <mesh filename="file://$(find dji_m600_sim)/meshes/m600.dae" scale="${chassisScale} ${chassisScale} ${chassisScale}"/>
-        </geometry>
-        <origin rpy="0 0 0" xyz="${chassisMeshXoffset} ${chassisMeshYoffset} ${chassisMeshZoffset}" />
-        <!-- <material name="blue" /> -->
+        <!-- <geometry> -->
+          <!-- <mesh filename="file://$(find dji_m600_sim)/meshes/m600.dae" scale="${chassisScale} ${chassisScale} ${chassisScale}"/> -->
+        <!-- </geometry> -->
+        <!-- <origin rpy="0 0 0" xyz="${chassisMeshXoffset} ${chassisMeshYoffset} ${chassisMeshZoffset}" /> -->
+        <xacro:box_geometry />
+        <material name="blue" />
       </visual>
       <collision>

Commit message: Fixed visualization

File: dji_m600_sim/urdf/links.xacro (robot description, xacro)
@@ -9,17 +9,18 @@
   <xacro:macro name="base_link">
    <link name="world"/>
-    <joint name="base_joint" type="fixed">
+   <link name="base_link"/>
+    <joint name="vehicle_center_joint" type="fixed">
       <parent link="world"/>
-      <child link="base_link" />
+      <child link="vehicle_center_link" />
       <origin xyz="${chassisXoffset} ${chassisYoffset} ${chassisZoffset}" rpy="0 0 0"/>
     </joint>
-    <link name="base_link">
+    <link name="vehicle_center_link">
       <visual>
-        <!-- <geometry> -->
-          <!-- <mesh filename="file://$(find dji_m600_sim)/meshes/m600.dae" scale="${chassisScale} ${chassisScale} ${chassisScale}"/> -->
-        <!-- </geometry> -->
-        <!-- <origin rpy="0 0 0" xyz="${chassisMeshXoffset} ${chassisMeshYoffset} ${chassisMeshZoffset}" /> -->
-        <xacro:box_geometry />
-        <material name="blue" />
+        <geometry>
+          <mesh filename="file://$(find dji_m600_sim)/meshes/m600.dae" scale="${chassisScale} ${chassisScale} ${chassisScale}"/>
+        </geometry>
+        <origin rpy="0 0 0" xyz="${chassisMeshXoffset} ${chassisMeshYoffset} ${chassisMeshZoffset}" />
+        <!-- <xacro:box_geometry /> -->
+        <!-- <material name="blue" /> -->
       </visual>
       <collision>
@@ -28,4 +29,9 @@
       <xacro:box_inertial/>
     </link>
+    <joint name="vehicle_ground_joint" type="fixed">
+      <parent link="vehicle_center_link"/>
+      <child link="base_link" />
+      <origin xyz="0 0 -${chassisZoffset}" rpy="0 0 0"/>
+    </joint>
     <xacro:base_gazebo/>
   </xacro:macro>

File: dji_m600_sim/urdf/properties.xacro (robot description, xacro)
@@ -8,5 +8,5 @@
     <xacro:property name="chassisXoffset" value="0.0" />
     <xacro:property name="chassisYoffset" value="0.0" />
-    <xacro:property name="chassisZoffset" value="${0.5*chassisH}" />
+    <xacro:property name="chassisZoffset" value="0.55" />
     <xacro:property name="chassisMass" value="1"/>
     <xacro:property name="chassisIxx" value="0.4"/>
@@ -19,4 +19,4 @@
     <xacro:property name="chassisMeshXoffset" value="0.000"/>
     <xacro:property name="chassisMeshYoffset" value="0.000"/>
-    <xacro:property name="chassisMeshZoffset" value="-0.36"/>
+    <xacro:property name="chassisMeshZoffset" value="-${chassisZoffset}"/>
 </robot>

Commit message: Refactor Packages

File: dji_m600_sim/urdf/links.xacro (robot description, xacro)
@@ -17,10 +17,10 @@
     <link name="vehicle_center_link">
       <visual>
-        <!-- <geometry> -->
-          <!-- <mesh filename="file://$(find dji_m600_sim)/meshes/m600.dae" scale="${chassisScale} ${chassisScale} ${chassisScale}"/> -->
-        <!-- </geometry> -->
+        <geometry>
+          <mesh filename="file://$(find dji_m600_sim)/meshes/m600.dae" scale="${chassisScale} ${chassisScale} ${chassisScale}"/>
+        </geometry>
         <origin rpy="0 0 0" xyz="${chassisMeshXoffset} ${chassisMeshYoffset} ${chassisMeshZoffset}" />
-        <xacro:drone_cylinder />
-        <material name="blue" />
+        <!-- <xacro:drone_cylinder /> -->
+        <!-- <material name="blue" /> -->
       </visual>
       <collision>
