Commit message: Perform HITL testing

File: dji_m600_sim/urdf/properties.xacro (robot description, xacro)
@@ -8,5 +8,6 @@
     <xacro:property name="chassisXoffset" value="0.0" />
     <xacro:property name="chassisYoffset" value="0.0" />
-    <xacro:property name="chassisZoffset" value="0.55" />
+    <xacro:property name="chassisZoffset" value="0.0" />
+    <!-- <xacro:property name="chassisZoffset" value="0.55" /> -->
     <xacro:property name="chassisMass" value="1"/>
     <xacro:property name="chassisIxx" value="0.4"/>
@@ -20,3 +21,4 @@
     <xacro:property name="chassisMeshYoffset" value="0.000"/>
     <xacro:property name="chassisMeshZoffset" value="-${chassisZoffset}"/>
+    <!-- <xacro:property name="chassisMeshZoffset" value="0.0"/>  -->
 </robot>
